Commit message: feat(vehicle): update vehicle dimensions, interface launch, and meshes

File: autobus_vehicle_description/urdf/vehicle.xacro (robot description, xacro)
@@ -3,10 +3,10 @@
   <!-- load parameter -->
   <xacro:property name="vehicle_info" value="${xacro.load_yaml('$(find autobus_vehicle_description)/config/vehicle_info.param.yaml')}"/>
-  <!-- vehicle body -->
+  <!-- vehicle body, no float need to find -->
   <link name="base_link">
     <visual>
-      <origin xyz="${vehicle_info['/**']['ros__parameters']['wheel_base']/2.0} 0 0" rpy="${pi/2.0} 0 ${pi}"/>
+      <origin xyz="1.27 -0.37 0" rpy="${pi/2.0} 0 ${pi}"/>
       <geometry>
-        <mesh filename="package://autobus_vehicle_description/mesh/lexus.dae" scale="1 1 1"/>
+        <mesh filename="package://autobus_vehicle_description/mesh/Full_Assem.STL" scale="0.001 0.001 0.001"/>
       </geometry>
     </visual>
